File: servo-drive/servo-drive.kicad_sch (KiCad schematic)
At the start: 53 parts, among them J1 SM04B-SRSS-TB, J10 Debug connector, J11 Conn_01x02, J12 Conn_01x02, J13 Conn_01x02, J14 Conn_01x02, J2 SM04B-SRSS-TB, J3 SM04B-SRSS-TB, J4 SM04B-SRSS-TB, J5 Battery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

Commit message: serial working!
Other:
- note added: "1.61 mA/count"
Changed lines of the file:
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@@
+		)
+	)
+	(text "1.61 mA/count"
+		(exclude_from_sim no)
+		(at 140.716 119.888 90)
+		(effects
+			(font
+				(size 1.27 1.27)
+			)
 		)
 	)
